Commit message: Bug 2 navigation package - submission ready
Co-Authored-By: Claude Opus 4.6 (1M context) <noreply@anthropic.com>

File: src/com760cw2_group5/urdf/group5Bot.urdf (robot description, URDF)
Before this commit: robot group5Bot, 5 links, 4 joints
Links:
- link base_link_chassis: geometry collision box size=0.2 0.15 0.05; visual box size=0.5 0.3 0.07
